Commit message: d
d

File: dfx_ground_robot_description/urdf/dfx_ground_robot.urdf (robot description, URDF)
Before this commit: robot dfx_ground_robot, 7 links, 6 joints
Joints:
- removed joint left front joint
- removed joint left rear joint
- removed joint right front joint
- removed joint right rear joint
- added joint left_front_joint: type continuous, parent base_link, child left_front_wheel, origin xyz=0.11 0.08 0.0, axis 1 0 0, limit lower=-3.14 upper=3.14 effort=300 velocity=0.1
- added joint left_rear_joint: type continuous, parent base_link, child left_rear_wheel, origin xyz=-0.11 0.08 0.0, axis 1 0 0, limit lower=-3.14 upper=3.14 effort=300 velocity=0.1
- added joint right_front_joint: type continuous, parent base_link, child right_front_wheel, origin xyz=0.11 -0.08 0.0, axis 1 0 0, limit lower=-3.14 upper=3.14 effort=300 velocity=0.1
- added joint right_rear_joint: type continuous, parent base_link, child right_rear_wheel, origin xyz=-0.11 -0.08 0.0, axis 1 0 0, limit lower=-3.14 upper=3.14 effort=300 velocity=0.1

File: dfx_ground_robot_description/urdf/dfx_ground_robot.xacro (robot description, xacro)
@@ -34,5 +34,5 @@
             </inertial>
     </link>
-    <joint name="right front joint" type="revolute">
+    <joint name="right_front_joint" type="continuous">
         <parent link="base_link"/>
         <child link="right_front_wheel"/>
@@ -64,5 +64,5 @@
         </inertial>
     </link>
-    <joint name="right rear joint" type="revolute">
+    <joint name="right_rear_joint" type="continuous">
         <parent link="base_link"/>
         <child link="right_rear_wheel"/>
@@ -94,5 +94,5 @@
         </inertial>
     </link>
-    <joint name="left front joint" type="revolute">
+    <joint name="left_front_joint" type="continuous">
         <parent link="base_link"/>
         <child link="left_front_wheel"/>
@@ -124,5 +124,5 @@
         </inertial>
     </link>
-    <joint name="left rear joint" type="revolute">
+    <joint name="left_rear_joint" type="continuous">
         <parent link="base_link"/>
         <child link="left_rear_wheel"/>
